Commit message: M6收尾，M7开端

File: src/ur_simulation_gz/ur_simulation_gz/urdf/multi_arm_robot.xacro (robot description, xacro)
@@ -1,7 +1,13 @@
 <?xml version="1.0"?>
 <!--
-  multi_arm_robot.xacro
-  Combined dual-arm URDF for MoveIt2 planning.
-  arm1_/arm2_ prefix, single CM, arm2 offset x=1.0m
+  multi_arm_robot.xacro — Backward-compatible wrapper for robot.xacro (M7.0.1).
+  This file is kept for backward compatibility with existing launch files and
+  config files that reference "multi_arm_robot.xacro".
+  The actual robot definition is now in robot.xacro (modular assembly).
+  Existing references (do not change):
+    - src/multi_arm_simulation/launch/*.launch.py
+    - src/multi_arm_moveit_config/launch/*.launch.py
+    - src/multi_arm_robot_description/config/robot.yaml
+    - src/multi_arm_simulation/config/hardware_adapters.yaml
 -->
 <robot xmlns:xacro="http://www.ros.org/wiki/xacro" name="multi_arm">
@@ -9,150 +15,4 @@
   <xacro:arg name="ur_type" default="ur5e"/>
   <xacro:arg name="simulation_controllers" default=""/>
-  <xacro:arg name="joint_limit_params"
-    default="$(find ur_description)/config/$(arg ur_type)/joint_limits.yaml"/>
-  <xacro:arg name="kinematics_params"
-    default="$(find ur_description)/config/$(arg ur_type)/default_kinematics.yaml"/>
-  <xacro:arg name="physical_params"
-    default="$(find ur_description)/config/$(arg ur_type)/physical_parameters.yaml"/>
-  <xacro:arg name="visual_params"
-    default="$(find ur_description)/config/$(arg ur_type)/visual_parameters.yaml"/>
-  <xacro:include filename="$(find ur_description)/urdf/ur_macro.xacro"/>
-  <!-- World root -->
-  <link name="world"/>
-  <link name="base_link">
-    <visual>
-      <origin xyz="0.5 0 0" rpy="0 0 0"/>
-      <geometry><box size="1.6 0.6 0.05"/></geometry>
-      <material name="base_plate"><color rgba="0.6 0.6 0.6 0.8"/></material>
-    </visual>
-    <collision>
-      <origin xyz="0.5 0 0" rpy="0 0 0"/>
-      <geometry><box size="1.6 0.6 0.05"/></geometry>
-    </collision>
-    <inertial>
-      <mass value="10.0"/>
-      <origin xyz="0.5 0 0" rpy="0 0 0"/>
-      <inertia ixx="0.1" ixy="0" ixz="0" iyy="0.1" iyz="0" izz="0.1"/>
-    </inertial>
-  </link>
-  <joint name="world_to_base" type="fixed">
-    <origin xyz="0 0 0" rpy="0 0 0"/>
-    <parent link="world"/>
-    <child link="base_link"/>
-  </joint>
-  <!-- arm1: mounted at base_link origin -->
-  <xacro:ur_robot
-    name="$(arg name)"
-    tf_prefix="arm1_"
-    parent="base_link"
-    joint_limits_parameters_file="$(arg joint_limit_params)"
-    kinematics_parameters_file="$(arg kinematics_params)"
-    physical_parameters_file="$(arg physical_params)"
-    visual_parameters_file="$(arg visual_params)"
-    safety_limits="true"
-    safety_pos_margin="0.15"
-    safety_k_position="20"
-    force_abs_paths="true">
-    <origin xyz="0 0 0" rpy="0 0 0"/>
-  </xacro:ur_robot>
-  <!-- arm2: mounted at x=1.0m offset -->
-  <xacro:ur_robot
-    name="$(arg name)"
-    tf_prefix="arm2_"
-    parent="base_link"
-    joint_limits_parameters_file="$(arg joint_limit_params)"
-    kinematics_parameters_file="$(arg kinematics_params)"
-    physical_parameters_file="$(arg physical_params)"
-    visual_parameters_file="$(arg visual_params)"
-    safety_limits="true"
-    safety_pos_margin="0.15"
-    safety_k_position="20"
-    force_abs_paths="true">
-    <origin xyz="1.0 0 0" rpy="0 0 0"/>
-  </xacro:ur_robot>
-  <!-- Gazebo plugin -->
-  <gazebo reference="world"/>
-  <gazebo>
-    <plugin filename="gz_ros2_control-system" name="gz_ros2_control::GazeboSimROS2ControlPlugin">
-      <parameters>$(arg simulation_controllers)</parameters>
-    </plugin>
-  </gazebo>
-  <!-- ros2_control (12 joints) -->
-  <ros2_control name="MultiArmSystem" type="system">
-    <hardware>
-      <plugin>gz_ros2_control/GazeboSimSystem</plugin>
-    </hardware>
-    <joint name="arm1_shoulder_pan_joint">
-      <command_interface name="position"/>
-      <state_interface name="position"><param name="initial_value">0.0</param></state_interface>
-      <state_interface name="velocity"><param name="initial_value">0.0</param></state_interface>
-      <state_interface name="effort"><param name="initial_value">0.0</param></state_interface>
-    </joint>
-    <joint name="arm1_shoulder_lift_joint">
-      <command_interface name="position"/>
-      <state_interface name="position"><param name="initial_value">-1.57</param></state_interface>
-      <state_interface name="velocity"><param name="initial_value">0.0</param></state_interface>
-      <state_interface name="effort"><param name="initial_value">0.0</param></state_interface>
-    </joint>
-    <joint name="arm1_elbow_joint">
-      <command_interface name="position"/>
-      <state_interface name="position"><param name="initial_value">0.0</param></state_interface>
-      <state_interface name="velocity"><param name="initial_value">0.0</param></state_interface>
-      <state_interface name="effort"><param name="initial_value">0.0</param></state_interface>
-    </joint>
-    <joint name="arm1_wrist_1_joint">
-      <command_interface name="position"/>
-      <state_interface name="position"><param name="initial_value">-1.57</param></state_interface>
-      <state_interface name="velocity"><param name="initial_value">0.0</param></state_interface>
-      <state_interface name="effort"><param name="initial_value">0.0</param></state_interface>
-    </joint>
-    <joint name="arm1_wrist_2_joint">
-      <command_interface name="position"/>
-      <state_interface name="position"><param name="initial_value">0.0</param></state_interface>
-      <state_interface name="velocity"><param name="initial_value">0.0</param></state_interface>
-      <state_interface name="effort"><param name="initial_value">0.0</param></state_interface>
-    </joint>
-    <joint name="arm1_wrist_3_joint">
-      <command_interface name="position"/>
-      <state_interface name="position"><param name="initial_value">0.0</param></state_interface>
-      <state_interface name="velocity"><param name="initial_value">0.0</param></state_interface>
-      <state_interface name="effort"><param name="initial_value">0.0</param></state_interface>
-    </joint>
-    <joint name="arm2_shoulder_pan_joint">
-      <command_interface name="position"/>
-      <state_interface name="position"><param name="initial_value">0.0</param></state_interface>
-      <state_interface name="velocity"><param name="initial_value">0.0</param></state_interface>
-      <state_interface name="effort"><param name="initial_value">0.0</param></state_interface>
-    </joint>
-    <joint name="arm2_shoulder_lift_joint">
-      <command_interface name="position"/>
-      <state_interface name="position"><param name="initial_value">-1.57</param></state_interface>
-      <state_interface name="velocity"><param name="initial_value">0.0</param></state_interface>
-      <state_interface name="effort"><param name="initial_value">0.0</param></state_interface>
-    </joint>
-    <joint name="arm2_elbow_joint">
-      <command_interface name="position"/>
-      <state_interface name="position"><param name="initial_value">0.0</param></state_interface>
-      <state_interface name="velocity"><param name="initial_value">0.0</param></state_interface>
-      <state_interface name="effort"><param name="initial_value">0.0</param></state_interface>
-    </joint>
-    <joint name="arm2_wrist_1_joint">
-      <command_interface name="position"/>
-      <state_interface name="position"><param name="initial_value">-1.57</param></state_interface>
-      <state_interface name="velocity"><param name="initial_value">0.0</param></state_interface>
-      <state_interface name="effort"><param name="initial_value">0.0</param></state_interface>
-    </joint>
-    <joint name="arm2_wrist_2_joint">
-      <command_interface name="position"/>
-      <state_interface name="position"><param name="initial_value">0.0</param></state_interface>
-      <state_interface name="velocity"><param name="initial_value">0.0</param></state_interface>
-      <state_interface name="effort"><param name="initial_value">0.0</param></state_interface>
-    </joint>
-    <joint name="arm2_wrist_3_joint">
-      <command_interface name="position"/>
-      <state_interface name="position"><param name="initial_value">0.0</param></state_interface>
-      <state_interface name="velocity"><param name="initial_value">0.0</param></state_interface>
-      <state_interface name="effort"><param name="initial_value">0.0</param></state_interface>
-    </joint>
-  </ros2_control>
+  <xacro:include filename="$(find ur_simulation_gz)/urdf/robot.xacro"/>
 </robot>
