Commit message: phase2.5: LED status binding to runtime state
- New led_status_node in multi_arm_runtime_api:
  - Checks /safety/check service and /execute_task action availability
  - States: INITIALIZING -> READY / FAILED / SAFETY_STOP
  - Publishes /led/status (std_msgs/String) and /led/color (std_msgs/ColorRGBA)
  - SAFETY_STOP flashes red
- New materials: led_red, led_blue, led_off in materials.xacro
- Launch file: led_status.launch.py
- Design doc updated: head_led_ring_link removed (replaced by head_depth_link in Phase 2.1)

Tests: 12 LED status tests + 27 URDF tests pass

File: src/ur_simulation_gz/ur_simulation_gz/urdf/materials.xacro (robot description, xacro)
@@ -7,4 +7,7 @@
   <material name="wheel_black"><color rgba="0.05 0.05 0.05 1.0"/></material>
   <material name="led_green"><color rgba="0.0 0.8 0.0 1.0"/></material>
+  <material name="led_red"><color rgba="0.8 0.0 0.0 1.0"/></material>
+  <material name="led_blue"><color rgba="0.0 0.0 0.8 1.0"/></material>
+  <material name="led_off"><color rgba="0.1 0.1 0.1 1.0"/></material>
   <material name="torso_white"><color rgba="0.8 0.8 0.8 1.0"/></material>
   <material name="head_dark"><color rgba="0.15 0.15 0.15 1.0"/></material>
