Commit message: M7阶段完成

File: src/ur_simulation_gz/ur_simulation_gz/urdf/body/head.xacro (robot description, xacro)
@@ -1,16 +1,71 @@
 <?xml version="1.0"?>
 <!--
-  head.xacro — Head module placeholder for M7.1 Robot Body Upgrade.
-  M7.0.1: Placeholder (no head, perception uses wrist camera only).
-  M7.1: Will add head (pan-tilt) with head-mounted camera for attention control.
-  Note: head_controller is separate from torso_controller.
+  head.xacro — Head module (M7.1 Robot Body Upgrade).
+  Adds neck_pitch_joint (revolute Y) between parent_link and head_link,
+  plus head_camera_link with RGB-D camera for perception attention.
+  head_controller is separate from torso_controller.
   Head belongs to Perception Attention System, not manipulation chain.
   Params:
-    parent_link  - link to mount head on (default "base_link")
+    parent_link  - link to mount head on (default "torso_link")
 -->
 <robot xmlns:xacro="http://www.ros.org/wiki/xacro">
-  <xacro:macro name="head" params="parent_link:='base_link'">
-    <!-- M7.1: Head (pan-tilt 2-DOF) + head camera will be added here -->
-    <!-- Placeholder: no-op macro, perception uses wrist camera in M7.0 -->
+  <xacro:macro name="head" params="parent_link:='torso_link'">
+    <link name="head_link">
+      <visual>
+        <origin xyz="0 0 0.05" rpy="0 0 0"/>
+        <geometry><box size="0.12 0.18 0.1"/></geometry>
+        <material name="panel_dark"/>
+      </visual>
+      <collision>
+        <origin xyz="0 0 0.05" rpy="0 0 0"/>
+        <geometry><box size="0.12 0.18 0.1"/></geometry>
+      </collision>
+      <inertial>
+        <mass value="1.5"/>
+        <origin xyz="0 0 0.05" rpy="0 0 0"/>
+        <inertia ixx="0.01" ixy="0" ixz="0" iyy="0.01" iyz="0" izz="0.01"/>
+      </inertial>
+    </link>
+    <joint name="neck_pitch_joint" type="revolute">
+      <origin xyz="0.5 0 0.85" rpy="0 0 0"/>
+      <parent link="${parent_link}"/>
+      <child link="head_link"/>
+      <axis xyz="0 1 0"/>
+      <limit lower="-1.57" upper="1.57" effort="10.0" velocity="0.5"/>
+    </joint>
+    <link name="head_camera_link">
+      <visual>
+        <origin xyz="0.05 0 0" rpy="0 1.5708 0"/>
+        <geometry><cylinder length="0.04" radius="0.03"/></geometry>
+        <material name="panel_dark"/>
+      </visual>
+      <inertial>
+        <mass value="0.2"/>
+        <inertia ixx="0.001" ixy="0" ixz="0" iyy="0.001" iyz="0" izz="0.001"/>
+      </inertial>
+    </link>
+    <joint name="head_to_camera" type="fixed">
+      <origin xyz="0.06 0 0.05" rpy="0 0 0"/>
+      <parent link="head_link"/>
+      <child link="head_camera_link"/>
+    </joint>
+    <gazebo reference="head_camera_link">
+      <sensor name="head_camera" type="rgbd">
+        <camera>
+          <horizontal_fov>1.5708</horizontal_fov>
+          <image>
+            <width>1280</width>
+            <height>720</height>
+          </image>
+          <clip>
+            <near>0.1</near>
+            <far>20.0</far>
+          </clip>
+        </camera>
+        <always_on>1</always_on>
+        <update_rate>30</update_rate>
+        <topic>head_camera/image_raw</topic>
+      </sensor>
+    </gazebo>
   </xacro:macro>
 </robot>

File: src/ur_simulation_gz/ur_simulation_gz/urdf/body/torso.xacro (robot description, xacro)
@@ -1,7 +1,8 @@
 <?xml version="1.0"?>
 <!--
-  torso.xacro — Torso module placeholder for M7.1 Robot Body Upgrade.
-  M7.0.1: Placeholder (no torso, arms mount directly on base pillars).
-  M7.1: Will add adjustable torso (1-DOF height) between base and arm pillars.
+  torso.xacro — Torso module (M7.1 Robot Body Upgrade).
+  Adds torso_yaw_joint (revolute Z) between base_link and torso_link.
+  Arms remain on base pillars; torso provides body rotation for
+  workspace expansion and IMU mounting point.
   Params:
     parent_link  - base link to mount torso on (default "base_link")
@@ -9,6 +10,27 @@
 <robot xmlns:xacro="http://www.ros.org/wiki/xacro">
   <xacro:macro name="torso" params="parent_link:='base_link'">
-    <!-- M7.1: Adjustable torso (1-DOF prismatic) will be added here -->
-    <!-- Placeholder: no-op macro, arms mount directly on base pillars in M7.0 -->
+    <link name="torso_link">
+      <visual>
+        <origin xyz="0.5 0 0.55" rpy="0 0 0"/>
+        <geometry><cylinder length="0.5" radius="0.15"/></geometry>
+        <material name="pillar_gray"/>
+      </visual>
+      <collision>
+        <origin xyz="0.5 0 0.55" rpy="0 0 0"/>
+        <geometry><cylinder length="0.5" radius="0.15"/></geometry>
+      </collision>
+      <inertial>
+        <mass value="8.0"/>
+        <origin xyz="0.5 0 0.55" rpy="0 0 0"/>
+        <inertia ixx="0.2" ixy="0" ixz="0" iyy="0.2" iyz="0" izz="0.1"/>
+      </inertial>
+    </link>
+    <joint name="torso_yaw_joint" type="revolute">
+      <origin xyz="0 0 0.3" rpy="0 0 0"/>
+      <parent link="${parent_link}"/>
+      <child link="torso_link"/>
+      <axis xyz="0 0 1"/>
+      <limit lower="-3.14" upper="3.14" effort="50.0" velocity="1.0"/>
+    </joint>
   </xacro:macro>
 </robot>

File: src/ur_simulation_gz/ur_simulation_gz/urdf/robot.xacro (robot description, xacro)
@@ -42,8 +42,8 @@
   <!-- 1. Mobile base (chassis + wheels + arm pillars) -->
   <xacro:wheeled_base prefix=""/>
-  <!-- 2. Torso (M7.0 placeholder: no-op, arms mount on pillars) -->
+  <!-- 2. Torso (M7.1: torso_yaw_joint revolute Z on base_link) -->
   <xacro:torso parent_link="base_link"/>
-  <!-- 3. Head (M7.0 placeholder: no-op, perception uses wrist camera) -->
-  <xacro:head parent_link="base_link"/>
+  <!-- 3. Head (M7.1: neck_pitch_joint revolute Y on torso_link + RGB-D) -->
+  <xacro:head parent_link="torso_link"/>
   <!-- 4. Dual UR5e arms + grippers -->
   <xacro:dual_ur5e
@@ -60,6 +60,6 @@
     sensor_name="arm1_wrist_camera"
     topic="arm1/camera/image_raw"/>
-  <xacro:imu_sensor parent_link="base_link" sensor_name="base_imu"/>
-  <!-- 6. ros2_control (14 joints: 12 arm + 2 gripper) -->
+  <xacro:imu_sensor parent_link="torso_link" sensor_name="torso_imu"/>
+  <!-- 6. ros2_control (16 joints: 12 arm + 2 gripper + 1 torso + 1 head) -->
   <xacro:multi_arm_ros2_control controllers_file="$(arg simulation_controllers)"/>
 </robot>

File: src/ur_simulation_gz/ur_simulation_gz/urdf/ros2_control/multi_arm_ros2_control.xacro (robot description, xacro)
@@ -1,6 +1,6 @@
 <?xml version="1.0"?>
 <!--
-  multi_arm_ros2_control.xacro — ros2_control block for dual-arm + grippers.
-  14 joints: 6 (arm1) + 6 (arm2) + 1 (arm1 gripper) + 1 (arm2 gripper).
+  multi_arm_ros2_control.xacro — ros2_control block for dual-arm + grippers + torso + head.
+  16 joints: 6 (arm1) + 6 (arm2) + 1 (arm1 gripper) + 1 (arm2 gripper) + 1 (torso) + 1 (head).
   GazeboSimSystem hardware plugin for Gazebo simulation.
   Params:
@@ -15,9 +15,23 @@
       </plugin>
     </gazebo>
-    <!-- ros2_control (14 joints: 12 arm + 2 gripper) -->
+    <!-- ros2_control (16 joints: 12 arm + 2 gripper + 1 torso + 1 head) -->
     <ros2_control name="MultiArmSystem" type="system">
       <hardware>
         <plugin>gz_ros2_control/GazeboSimSystem</plugin>
       </hardware>
+      <!-- torso joint (1 DOF, Z yaw) -->
+      <joint name="torso_yaw_joint">
+        <command_interface name="position"/>
+        <state_interface name="position"><param name="initial_value">0.0</param></state_interface>
+        <state_interface name="velocity"><param name="initial_value">0.0</param></state_interface>
+        <state_interface name="effort"><param name="initial_value">0.0</param></state_interface>
+      </joint>
+      <!-- head joint (1 DOF, Y pitch) -->
+      <joint name="neck_pitch_joint">
+        <command_interface name="position"/>
+        <state_interface name="position"><param name="initial_value">0.0</param></state_interface>
+        <state_interface name="velocity"><param name="initial_value">0.0</param></state_interface>
+        <state_interface name="effort"><param name="initial_value">0.0</param></state_interface>
+      </joint>
       <!-- arm1 joints (6 DOF) -->
       <joint name="arm1_shoulder_pan_joint">

File: src/ur_simulation_gz/ur_simulation_gz/urdf/sensors/imu.xacro (robot description, xacro)
@@ -1,17 +1,22 @@
 <?xml version="1.0"?>
 <!--
-  imu.xacro — IMU sensor placeholder for M7.4 Perception+Calibration.
-  M7.0.1: Placeholder only (no physical IMU yet).
-  M7.4: Will add real IMU sensor on base_link for odometry fusion.
+  imu.xacro — IMU sensor (M7.1 Robot Body Upgrade).
+  Gazebo IMU sensor on torso_link for body attitude estimation.
+  IMU is on torso, not head — torso attitude is the body attitude.
   Params:
-    parent_link  - link to attach IMU to (default "base_link")
-    sensor_name  - sensor name (default "base_imu")
+    parent_link  - link to attach IMU to (default "torso_link")
+    sensor_name  - sensor name (default "torso_imu")
     rate         - update rate Hz (default 100)
 -->
 <robot xmlns:xacro="http://www.ros.org/wiki/xacro">
   <xacro:macro name="imu_sensor"
-    params="parent_link:='base_link' sensor_name:='base_imu' rate:=100">
-    <!-- M7.4: Real IMU sensor will be added here -->
-    <!-- Placeholder: no-op macro, expanded when M7.4 implements perception -->
+    params="parent_link:='torso_link' sensor_name:='torso_imu' rate:=100">
+    <gazebo reference="${parent_link}">
+      <sensor name="${sensor_name}" type="imu">
+        <always_on>1</always_on>
+        <update_rate>${rate}</update_rate>
+        <topic>${sensor_name}/data</topic>
+      </sensor>
+    </gazebo>
   </xacro:macro>
 </robot>

Commit message: 架构转变

File: src/ur_simulation_gz/ur_simulation_gz/urdf/body/head.xacro (robot description, xacro)
@@ -14,5 +14,7 @@
       <visual>
         <origin xyz="0 0 0.05" rpy="0 0 0"/>
-        <geometry><box size="0.12 0.18 0.1"/></geometry>
+        <geometry>
+          <box size="0.12 0.18 0.1"/>
+        </geometry>
         <material name="panel_dark"/>
       </visual>
@@ -37,6 +39,8 @@
       <visual>
         <origin xyz="0.05 0 0" rpy="0 1.5708 0"/>
-        <geometry><cylinder length="0.04" radius="0.03"/></geometry>
-        <material name="panel_dark"/>
+        <geometry>
+          <cylinder length="0.03" radius="0.012"/>
+        </geometry>
+        <material name="camera_lens"/>
       </visual>
       <inertial>
@@ -49,4 +53,22 @@
       <parent link="head_link"/>
       <child link="head_camera_link"/>
+    </joint>
+    <link name="head_led_ring_link">
+      <visual>
+        <origin xyz="0.05 0 0.05" rpy="1.5708 0 0"/>
+        <geometry>
+          <cylinder length="0.005" radius="0.03"/>
+        </geometry>
+        <material name="led_ring"/>
+      </visual>
+      <inertial>
+        <mass value="0.05"/>
+        <inertia ixx="0.0001" ixy="0" ixz="0" iyy="0.0001" iyz="0" izz="0.0001"/>
+      </inertial>
+    </link>
+    <joint name="head_to_led_ring" type="fixed">
+      <origin xyz="0 0 0" rpy="0 0 0"/>
+      <parent link="head_link"/>
+      <child link="head_led_ring_link"/>
     </joint>
     <gazebo reference="head_camera_link">

File: src/ur_simulation_gz/ur_simulation_gz/urdf/body/torso.xacro (robot description, xacro)
@@ -13,5 +13,7 @@
       <visual>
         <origin xyz="0.5 0 0.55" rpy="0 0 0"/>
-        <geometry><cylinder length="0.5" radius="0.15"/></geometry>
+        <geometry>
+          <cylinder length="0.5" radius="0.15"/>
+        </geometry>
         <material name="pillar_gray"/>
       </visual>

File: src/ur_simulation_gz/ur_simulation_gz/urdf/materials.xacro (robot description, xacro)
@@ -9,3 +9,8 @@
   <material name="torso_white"><color rgba="0.8 0.8 0.8 1.0"/></material>
   <material name="head_dark"><color rgba="0.15 0.15 0.15 1.0"/></material>
+  <material name="camera_lens"><color rgba="0.05 0.05 0.05 1.0"/></material>
+  <material name="led_ring"><color rgba="0.0 0.6 1.0 1.0"/></material>
+  <material name="display_panel"><color rgba="0.0 0.0 0.0 0.85"/></material>
+  <material name="metal_dark"><color rgba="0.2 0.2 0.22 1.0"/></material>
+  <material name="metal_light"><color rgba="0.7 0.7 0.72 1.0"/></material>
 </robot>

File: src/ur_simulation_gz/ur_simulation_gz/urdf/mobile_base/wheeled_base.xacro (robot description, xacro)
@@ -32,5 +32,7 @@
       <visual>
         <origin xyz="0.5 0 0.15" rpy="0 0 0"/>
-        <geometry><box size="1.4 0.5 0.3"/></geometry>
+        <geometry>
+          <box size="1.4 0.5 0.3"/>
+        </geometry>
         <material name="chassis_blue"/>
       </visual>
@@ -72,5 +74,7 @@
     <link name="status_led">
       <visual>
-        <geometry><box size="0.3 0.03 0.02"/></geometry>
+        <geometry>
+          <box size="1.0 0.01 0.02"/>
+        </geometry>
         <material name="led_green"/>
       </visual>
@@ -85,5 +89,7 @@
       <visual>
         <origin xyz="0 0 0.1" rpy="0 0 0"/>
-        <geometry><cylinder length="0.2" radius="0.08"/></geometry>
+        <geometry>
+          <cylinder length="0.2" radius="0.08"/>
+        </geometry>
         <material name="pillar_gray"/>
       </visual>
@@ -107,5 +113,7 @@
       <visual>
         <origin xyz="0 0 0.1" rpy="0 0 0"/>
-        <geometry><cylinder length="0.2" radius="0.08"/></geometry>
+        <geometry>
+          <cylinder length="0.2" radius="0.08"/>
+        </geometry>
         <material name="pillar_gray"/>
       </visual>
