Commit message: phase2(m2): xacro chain arm1/arm2 -> left_arm/right_arm
dual_ur5e.xacro: tf_prefix + parent + robotiq prefix
wheeled_base.xacro: pillar link/joint (arm1_pillar -> left_arm_pillar)
robot.xacro: wrist camera prefix/parent/topic
multi_arm_ros2_control.xacro: 12 arm joints + 2 gripper joints
robotiq_2f_85.xacro + camera.xacro: doc examples

6 files, 0 arm1/arm2 residual, XML valid, joint prefix consistent
Two URDF paths aligned: robot.yaml.prefix == dual_ur5e.xacro tf_prefix

File: src/ur_simulation_gz/ur_simulation_gz/urdf/arms/dual_ur5e.xacro (robot description, xacro)
@@ -2,5 +2,5 @@
 <!--
   dual_ur5e.xacro — Dual UR5e arms with Robotiq 2F-85 grippers.
-  Instantiates two UR5e arms on arm1_pillar / arm2_pillar,
+  Instantiates two UR5e arms on left_arm_pillar / right_arm_pillar,
   each with a Robotiq 2F-85 gripper on tool0.
   Params:
@@ -17,9 +17,9 @@
   <xacro:macro name="dual_ur5e"
     params="name ur_type joint_limit_params kinematics_params physical_params visual_params">
-    <!-- arm1: mounted on arm1_pillar -->
+    <!-- left_arm: mounted on left_arm_pillar -->
     <xacro:ur_robot
       name="${name}"
-      tf_prefix="arm1_"
-      parent="arm1_pillar"
+      tf_prefix="left_arm_"
+      parent="left_arm_pillar"
       joint_limits_parameters_file="${joint_limit_params}"
       kinematics_parameters_file="${kinematics_params}"
@@ -32,11 +32,11 @@
       <origin xyz="0 0 0.2" rpy="0 0 0"/>
     </xacro:ur_robot>
-    <!-- arm1: Robotiq 2F-85 gripper -->
-    <xacro:robotiq_2f_85 prefix="arm1_" parent="arm1_tool0"/>
-    <!-- arm2: mounted on arm2_pillar -->
+    <!-- left_arm: Robotiq 2F-85 gripper -->
+    <xacro:robotiq_2f_85 prefix="left_arm_" parent="left_arm_tool0"/>
+    <!-- right_arm: mounted on right_arm_pillar -->
     <xacro:ur_robot
       name="${name}"
-      tf_prefix="arm2_"
-      parent="arm2_pillar"
+      tf_prefix="right_arm_"
+      parent="right_arm_pillar"
       joint_limits_parameters_file="${joint_limit_params}"
       kinematics_parameters_file="${kinematics_params}"
@@ -49,6 +49,6 @@
       <origin xyz="0 0 0.2" rpy="0 0 0"/>
     </xacro:ur_robot>
-    <!-- arm2: Robotiq 2F-85 gripper -->
-    <xacro:robotiq_2f_85 prefix="arm2_" parent="arm2_tool0"/>
+    <!-- right_arm: Robotiq 2F-85 gripper -->
+    <xacro:robotiq_2f_85 prefix="right_arm_" parent="right_arm_tool0"/>
   </xacro:macro>
 </robot>

File: src/ur_simulation_gz/ur_simulation_gz/urdf/end_effectors/robotiq_2f_85.xacro (robot description, xacro)
@@ -4,6 +4,6 @@
   Simplified Robotiq 2F-85 parallel gripper for Gazebo simulation.
   Params:
-    prefix  - tf prefix (e.g. "arm1_")
-    parent  - parent link (e.g. "arm1_tool0")
+    prefix  - tf prefix (e.g. "left_arm_")
+    parent  - parent link (e.g. "left_arm_tool0")
 -->
 <robot xmlns:xacro="http://www.ros.org/wiki/xacro">

File: src/ur_simulation_gz/ur_simulation_gz/urdf/mobile_base/wheeled_base.xacro (robot description, xacro)
@@ -85,6 +85,6 @@
       <child link="status_led"/>
     </joint>
-    <!-- arm1 mounting pillar -->
-    <link name="arm1_pillar">
+    <!-- left_arm mounting pillar -->
+    <link name="left_arm_pillar">
       <visual>
         <origin xyz="0 0 0.1" rpy="0 0 0"/>
@@ -104,11 +104,11 @@
       </inertial>
     </link>
-    <joint name="base_to_arm1_pillar" type="fixed">
+    <joint name="base_to_left_arm_pillar" type="fixed">
       <origin xyz="0 0 0.3" rpy="0 0 0"/>
       <parent link="${prefix}base_link"/>
-      <child link="arm1_pillar"/>
+      <child link="left_arm_pillar"/>
     </joint>
-    <!-- arm2 mounting pillar -->
-    <link name="arm2_pillar">
+    <!-- right_arm mounting pillar -->
+    <link name="right_arm_pillar">
       <visual>
         <origin xyz="0 0 0.1" rpy="0 0 0"/>
@@ -128,8 +128,8 @@
       </inertial>
     </link>
-    <joint name="base_to_arm2_pillar" type="fixed">
+    <joint name="base_to_right_arm_pillar" type="fixed">
       <origin xyz="1.0 0 0.3" rpy="0 0 0"/>
       <parent link="${prefix}base_link"/>
-      <child link="arm2_pillar"/>
+      <child link="right_arm_pillar"/>
     </joint>
     <!-- 4 wheels (fixed joint, M7.6 will make revolute) -->

File: src/ur_simulation_gz/ur_simulation_gz/urdf/robot.xacro (robot description, xacro)
@@ -56,8 +56,8 @@
   <!-- 5. Sensors -->
   <xacro:wrist_camera
-    prefix="arm1_"
-    parent_link="arm1_wrist_3_link"
-    sensor_name="arm1_wrist_camera"
-    topic="arm1/camera/image_raw"/>
+    prefix="left_arm_"
+    parent_link="left_arm_wrist_3_link"
+    sensor_name="left_arm_wrist_camera"
+    topic="left_arm/camera/image_raw"/>
   <xacro:imu_sensor parent_link="torso_link" sensor_name="torso_imu"/>
   <!-- 6. ros2_control (16 joints: 12 arm + 2 gripper + 1 torso + 1 head) -->

File: src/ur_simulation_gz/ur_simulation_gz/urdf/ros2_control/multi_arm_ros2_control.xacro (robot description, xacro)
@@ -2,5 +2,5 @@
 <!--
   multi_arm_ros2_control.xacro — ros2_control block for dual-arm + grippers + torso + head.
-  16 joints: 6 (arm1) + 6 (arm2) + 1 (arm1 gripper) + 1 (arm2 gripper) + 1 (torso) + 1 (head).
+  16 joints: 6 (left_arm) + 6 (right_arm) + 1 (left_arm gripper) + 1 (right_arm gripper) + 1 (torso) + 1 (head).
   GazeboSimSystem hardware plugin for Gazebo simulation.
   Params:
@@ -34,6 +34,6 @@
         <state_interface name="effort"><param name="initial_value">0.0</param></state_interface>
       </joint>
-      <!-- arm1 joints (6 DOF) -->
-      <joint name="arm1_shoulder_pan_joint">
+      <!-- left_arm joints (6 DOF) -->
+      <joint name="left_arm_shoulder_pan_joint">
         <command_interface name="position"/>
         <state_interface name="position"><param name="initial_value">0.0</param></state_interface>
@@ -41,5 +41,5 @@
         <state_interface name="effort"><param name="initial_value">0.0</param></state_interface>
       </joint>
-      <joint name="arm1_shoulder_lift_joint">
+      <joint name="left_arm_shoulder_lift_joint">
         <command_interface name="position"/>
         <state_interface name="position"><param name="initial_value">-1.57</param></state_interface>
@@ -47,5 +47,5 @@
         <state_interface name="effort"><param name="initial_value">0.0</param></state_interface>
       </joint>
-      <joint name="arm1_elbow_joint">
+      <joint name="left_arm_elbow_joint">
         <command_interface name="position"/>
         <state_interface name="position"><param name="initial_value">0.0</param></state_interface>
@@ -53,5 +53,5 @@
         <state_interface name="effort"><param name="initial_value">0.0</param></state_interface>
       </joint>
-      <joint name="arm1_wrist_1_joint">
+      <joint name="left_arm_wrist_1_joint">
         <command_interface name="position"/>
         <state_interface name="position"><param name="initial_value">-1.57</param></state_interface>
@@ -59,5 +59,5 @@
         <state_interface name="effort"><param name="initial_value">0.0</param></state_interface>
       </joint>
-      <joint name="arm1_wrist_2_joint">
+      <joint name="left_arm_wrist_2_joint">
         <command_interface name="position"/>
         <state_interface name="position"><param name="initial_value">0.0</param></state_interface>
@@ -65,5 +65,5 @@
         <state_interface name="effort"><param name="initial_value">0.0</param></state_interface>
       </joint>
-      <joint name="arm1_wrist_3_joint">
+      <joint name="left_arm_wrist_3_joint">
         <command_interface name="position"/>
         <state_interface name="position"><param name="initial_value">0.0</param></state_interface>
@@ -71,6 +71,6 @@
         <state_interface name="effort"><param name="initial_value">0.0</param></state_interface>
       </joint>
-      <!-- arm2 joints (6 DOF) -->
-      <joint name="arm2_shoulder_pan_joint">
+      <!-- right_arm joints (6 DOF) -->
+      <joint name="right_arm_shoulder_pan_joint">
         <command_interface name="position"/>
         <state_interface name="position"><param name="initial_value">0.0</param></state_interface>
@@ -78,5 +78,5 @@
         <state_interface name="effort"><param name="initial_value">0.0</param></state_interface>
       </joint>
-      <joint name="arm2_shoulder_lift_joint">
+      <joint name="right_arm_shoulder_lift_joint">
         <command_interface name="position"/>
         <state_interface name="position"><param name="initial_value">-1.57</param></state_interface>
@@ -84,5 +84,5 @@
         <state_interface name="effort"><param name="initial_value">0.0</param></state_interface>
       </joint>
-      <joint name="arm2_elbow_joint">
+      <joint name="right_arm_elbow_joint">
         <command_interface name="position"/>
         <state_interface name="position"><param name="initial_value">0.0</param></state_interface>
@@ -90,5 +90,5 @@
         <state_interface name="effort"><param name="initial_value">0.0</param></state_interface>
       </joint>
-      <joint name="arm2_wrist_1_joint">
+      <joint name="right_arm_wrist_1_joint">
         <command_interface name="position"/>
         <state_interface name="position"><param name="initial_value">-1.57</param></state_interface>
@@ -96,5 +96,5 @@
         <state_interface name="effort"><param name="initial_value">0.0</param></state_interface>
       </joint>
-      <joint name="arm2_wrist_2_joint">
+      <joint name="right_arm_wrist_2_joint">
         <command_interface name="position"/>
         <state_interface name="position"><param name="initial_value">0.0</param></state_interface>
@@ -102,5 +102,5 @@
         <state_interface name="effort"><param name="initial_value">0.0</param></state_interface>
       </joint>
-      <joint name="arm2_wrist_3_joint">
+      <joint name="right_arm_wrist_3_joint">
         <command_interface name="position"/>
         <state_interface name="position"><param name="initial_value">0.0</param></state_interface>
@@ -108,6 +108,6 @@
         <state_interface name="effort"><param name="initial_value">0.0</param></state_interface>
       </joint>
-      <!-- arm1 gripper joint (1 DOF, mimic drives the rest) -->
-      <joint name="arm1_robotiq_left_knuckle_joint">
+      <!-- left_arm gripper joint (1 DOF, mimic drives the rest) -->
+      <joint name="left_arm_robotiq_left_knuckle_joint">
         <command_interface name="position"/>
         <state_interface name="position"><param name="initial_value">0.0</param></state_interface>
@@ -115,6 +115,6 @@
         <state_interface name="effort"><param name="initial_value">0.0</param></state_interface>
       </joint>
-      <!-- arm2 gripper joint (1 DOF, mimic drives the rest) -->
-      <joint name="arm2_robotiq_left_knuckle_joint">
+      <!-- right_arm gripper joint (1 DOF, mimic drives the rest) -->
+      <joint name="right_arm_robotiq_left_knuckle_joint">
         <command_interface name="position"/>
         <state_interface name="position"><param name="initial_value">0.0</param></state_interface>

File: src/ur_simulation_gz/ur_simulation_gz/urdf/sensors/camera.xacro (robot description, xacro)
@@ -3,8 +3,8 @@
   camera.xacro — Wrist-mounted camera sensor for Gazebo.
   Params:
-    prefix       - tf prefix (e.g. "arm1_")
-    parent_link  - link to attach camera to (e.g. "arm1_wrist_3_link")
-    sensor_name  - sensor name (e.g. "arm1_wrist_camera")
-    topic        - image topic (e.g. "arm1/camera/image_raw")
+    prefix       - tf prefix (e.g. "left_arm_")
+    parent_link  - link to attach camera to (e.g. "left_arm_wrist_3_link")
+    sensor_name  - sensor name (e.g. "left_arm_wrist_camera")
+    topic        - image topic (e.g. "left_arm/camera/image_raw")
     width        - image width  (default 640)
     height       - image height (default 480)

Commit message: phase2: head sensor split + shoulder_mount introduction
Phase 2.1 - Head sensor split:
- head_camera_link -> head_rgb_link + head_depth_link + head_imu_link
- Remove torso_imu (IMU moved to head_imu_link on head)
- Gazebo sensors: head_rgb (camera) + head_depth (depth) + head_imu (imu)
- robot.yaml: head_camera -> head_rgb + head_depth, head_imu frame updated

Phase 2.2 - shoulder_mount introduction:
- New links: left_shoulder_mount + right_shoulder_mount (children of torso_link)
- Arms reparented: left_arm_pillar -> left_shoulder_mount, right_arm_pillar -> right_shoulder_mount
- Arms now follow torso rotation (kinematic change)
- Pillars remain in wheeled_base as structural elements

SRDF collision matrix:
- pillar<->arm pairs -> shoulder_mount<->arm pairs
- Added torso<->shoulder_mount pairs
- Added head<->head_depth_link, head<->head_imu_link pairs

Tests:
- test_modular_urdf.py: pillar assertions -> shoulder_mount, revolute count 20->22
- test_m7_1_body.py: head_camera/torso_imu assertions -> head_rgb/head_depth/head_imu

Verified: 18 packages build, 27 URDF tests + 8 M7.1 tests pass, xacro render 1636 lines

File: src/ur_simulation_gz/ur_simulation_gz/urdf/arms/dual_ur5e.xacro (robot description, xacro)
@@ -2,5 +2,5 @@
 <!--
   dual_ur5e.xacro — Dual UR5e arms with Robotiq 2F-85 grippers.
-  Instantiates two UR5e arms on left_arm_pillar / right_arm_pillar,
+  Instantiates two UR5e arms on left_shoulder_mount / right_shoulder_mount,
   each with a Robotiq 2F-85 gripper on tool0.
   Params:
@@ -17,9 +17,9 @@
   <xacro:macro name="dual_ur5e"
     params="name ur_type joint_limit_params kinematics_params physical_params visual_params">
-    <!-- left_arm: mounted on left_arm_pillar -->
+    <!-- left_arm: mounted on left_shoulder_mount (torso_link) -->
     <xacro:ur_robot
       name="${name}"
       tf_prefix="left_arm_"
-      parent="left_arm_pillar"
+      parent="left_shoulder_mount"
       joint_limits_parameters_file="${joint_limit_params}"
       kinematics_parameters_file="${kinematics_params}"
@@ -34,9 +34,9 @@
     <!-- left_arm: Robotiq 2F-85 gripper -->
     <xacro:robotiq_2f_85 prefix="left_arm_" parent="left_arm_tool0"/>
-    <!-- right_arm: mounted on right_arm_pillar -->
+    <!-- right_arm: mounted on right_shoulder_mount (torso_link) -->
     <xacro:ur_robot
       name="${name}"
       tf_prefix="right_arm_"
-      parent="right_arm_pillar"
+      parent="right_shoulder_mount"
       joint_limits_parameters_file="${joint_limit_params}"
       kinematics_parameters_file="${kinematics_params}"

File: src/ur_simulation_gz/ur_simulation_gz/urdf/body/head.xacro (robot description, xacro)
@@ -3,5 +3,5 @@
   head.xacro — Head module (M7.1 Robot Body Upgrade).
   Adds neck_pitch_joint (revolute Y) between parent_link and head_link,
-  plus head_camera_link with RGB-D camera for perception attention.
+  plus head_rgb_link with RGB-D camera for perception attention.
   head_controller is separate from torso_controller.
   Head belongs to Perception Attention System, not manipulation chain.
@@ -36,5 +36,5 @@
       <limit lower="-1.57" upper="1.57" effort="10.0" velocity="0.5"/>
     </joint>
-    <link name="head_camera_link">
+    <link name="head_rgb_link">
       <visual>
         <origin xyz="0.05 0 0" rpy="0 1.5708 0"/>
@@ -46,32 +46,43 @@
       <inertial>
         <mass value="0.2"/>
-        <inertia ixx="0.001" ixy="0" ixz="0" iyy="0.001" iyz="0" izz="0.001"/>
+        <inertia ixx="0.001" ixy="0" ixz="0" iyy="0.001" yyz="0" izz="0.001"/>
       </inertial>
     </link>
-    <joint name="head_to_camera" type="fixed">
+    <joint name="head_to_rgb" type="fixed">
       <origin xyz="0.06 0 0.05" rpy="0 0 0"/>
       <parent link="head_link"/>
-      <child link="head_camera_link"/>
+      <child link="head_rgb_link"/>
     </joint>
-    <link name="head_led_ring_link">
+    <link name="head_depth_link">
       <visual>
-        <origin xyz="0.05 0 0.05" rpy="1.5708 0 0"/>
+        <origin xyz="0.05 0 0" rpy="0 1.5708 0"/>
         <geometry>
-          <cylinder length="0.005" radius="0.03"/>
+          <cylinder length="0.03" radius="0.012"/>
         </geometry>
-        <material name="led_ring"/>
+        <material name="camera_lens"/>
       </visual>
       <inertial>
-        <mass value="0.05"/>
-        <inertia ixx="0.0001" ixy="0" ixz="0" iyy="0.0001" iyz="0" izz="0.0001"/>
+        <mass value="0.2"/>
+        <inertia ixx="0.001" ixy="0" ixz="0" iyy="0.001" yyz="0" izz="0.001"/>
       </inertial>
     </link>
-    <joint name="head_to_led_ring" type="fixed">
+    <joint name="head_to_depth" type="fixed">
+      <origin xyz="0.11 0 0.05" rpy="0 0 0"/>
+      <parent link="head_link"/>
+      <child link="head_depth_link"/>
+    </joint>
+    <link name="head_imu_link">
+      <inertial>
+        <mass value="0.05"/>
+        <inertia ixx="0.0001" ixy="0" ixz="0" iyy="0.0001" yyz="0" izz="0.0001"/>
+      </inertial>
+    </link>
+    <joint name="head_to_imu" type="fixed">
       <origin xyz="0 0 0" rpy="0 0 0"/>
       <parent link="head_link"/>
-      <child link="head_led_ring_link"/>
+      <child link="head_imu_link"/>
     </joint>
-    <gazebo reference="head_camera_link">
-      <sensor name="head_camera" type="rgbd">
+    <gazebo reference="head_rgb_link">
+      <sensor name="head_rgb" type="camera">
         <camera>
           <horizontal_fov>1.5708</horizontal_fov>
@@ -87,5 +98,30 @@
         <always_on>1</always_on>
         <update_rate>30</update_rate>
-        <topic>head_camera/image_raw</topic>
+        <topic>head/rgb/image_raw</topic>
+      </sensor>
+    </gazebo>
+    <gazebo reference="head_depth_link">
+      <sensor name="head_depth" type="depth">
+        <camera>
+          <horizontal_fov>1.5708</horizontal_fov>
+          <image>
+            <width>1280</width>
+            <height>720</height>
+          </image>
+          <clip>
+            <near>0.1</near>
+            <far>20.0</far>
+          </clip>
+        </camera>
+        <always_on>1</always_on>
+        <update_rate>30</update_rate>
+        <topic>head/depth/image_raw</topic>
+      </sensor>
+    </gazebo>
+    <gazebo reference="head_imu_link">
+      <sensor name="head_imu" type="imu">
+        <always_on>1</always_on>
+        <update_rate>100</update_rate>
+        <topic>head/imu</topic>
       </sensor>
     </gazebo>

File: src/ur_simulation_gz/ur_simulation_gz/urdf/body/torso.xacro (robot description, xacro)
@@ -35,4 +35,26 @@
       <limit lower="-3.14" upper="3.14" effort="50.0" velocity="1.0"/>
     </joint>
+    <link name="left_shoulder_mount">
+      <inertial>
+        <mass value="0.5"/>
+        <inertia ixx="0.01" ixy="0" ixz="0" iyy="0.01" yyz="0" izz="0.01"/>
+      </inertial>
+    </link>
+    <joint name="torso_to_left_shoulder" type="fixed">
+      <origin xyz="0 0 0" rpy="0 0 0"/>
+      <parent link="torso_link"/>
+      <child link="left_shoulder_mount"/>
+    </joint>
+    <link name="right_shoulder_mount">
+      <inertial>
+        <mass value="0.5"/>
+        <inertia ixx="0.01" ixy="0" ixz="0" iyy="0.01" yyz="0" izz="0.01"/>
+      </inertial>
+    </link>
+    <joint name="torso_to_right_shoulder" type="fixed">
+      <origin xyz="1.0 0 0" rpy="0 0 0"/>
+      <parent link="torso_link"/>
+      <child link="right_shoulder_mount"/>
+    </joint>
   </xacro:macro>
 </robot>

File: src/ur_simulation_gz/ur_simulation_gz/urdf/robot.xacro (robot description, xacro)
@@ -60,5 +60,5 @@
     sensor_name="left_arm_wrist_camera"
     topic="left_arm/camera/image_raw"/>
-  <xacro:imu_sensor parent_link="torso_link" sensor_name="torso_imu"/>
+  <!-- IMU now in head.xacro (head_imu_link on head_link) -->
   <!-- 6. ros2_control (16 joints: 12 arm + 2 gripper + 1 torso + 1 head) -->
   <xacro:multi_arm_ros2_control controllers_file="$(arg simulation_controllers)"/>

File: src/ur_simulation_gz/ur_simulation_gz/urdf/sensors/imu.xacro (robot description, xacro)
@@ -6,10 +6,10 @@
   Params:
     parent_link  - link to attach IMU to (default "torso_link")
-    sensor_name  - sensor name (default "torso_imu")
+    sensor_name  - sensor name (default "head_imu")
     rate         - update rate Hz (default 100)
 -->
 <robot xmlns:xacro="http://www.ros.org/wiki/xacro">
   <xacro:macro name="imu_sensor"
-    params="parent_link:='torso_link' sensor_name:='torso_imu' rate:=100">
+    params="parent_link:='torso_link' sensor_name:='head_imu' rate:=100">
     <gazebo reference="${parent_link}">
       <sensor name="${sensor_name}" type="imu">
